File: VolToneEQ/VolToneEQ/VolToneEQ.sch (KiCad schematic (older format))
At the start: 6 parts

Commit message: Added most connections
Still needs EQ circuit and enough switches to cuf off both tone pots. might have to use 2 4pdts. Also make initial phase switches into one 4pdt.
Parts:
- added U? (x4): KEMET470p5mm, symbol 6mmKEMET:KEMET470p5mm
- added U?: 3WAYswitch, symbol 3WAY:3WAYswitch
- added U?: 6PDTswitch, symbol 6PDT:6PDTswitch
Connections:
- net labels added: BROUT, BVIN, BVINTRAD, BVOUT, BVOUTTRAD, GND, NOUT, NVIN, NVINTRAD, NVOUT, NVOUTTRAD, NWHITE, TOJACK
- net labels removed: BRBARE, NBARE
- wire segments 29 -> 161
Other:
- note added: "7,8,9 S1B (LEFT SIDE)\n\n10,11,12 S1A"
- note added: "7,8,9 S2A (LEFT SIDE)\n\n10,11,12 S2B"
- note added: "7,8,9 S3B (LEFT SIDE)\n\n10,11,12 S3A"
- note added: "7,8,9 S4A (LEFT SIDE)\n\n10,11,12 S4B"
- note added: "WIMA .022u 5mm"

Commit message: Updated LTSpice schematic with EQ
Parts:
- removed U?: 6PDTswitch, symbol 6PDT:6PDTswitch
- added U? (x2): 4pdtswitch, symbol 4pdt:4pdtswitch
Connections:
- net labels added: BTONE, BTONEIN, NTONE, NTONEIN
- wire segments 161 -> 157
Other:
- note added: "These 2 switches control traditional\nvs 3 band EQ selection"
Changed lines of the file:
@@
 L 4pdt:4pdtswitch U?
 U 1 1 5B812BE0
-P 4050 2350
-F 0 "U?" H 4450 2500 50  0000 C CNN
-F 1 "4pdtswitch" H 4450 2450 50  0000 C CNN
-F 2 "" H 4050 2350 50  0001 C CNN
-F 3 "" H 4050 2350 50  0001 C CNN
-	1    4050 2350
+P 4050 2450
+F 0 "U?" H 4300 2750 50  0000 C CNN
+F 1 "4pdtswitch" H 4300 2700 50  0000 C CNN
+F 2 "" H 4050 2450 50  0001 C CNN
+F 3 "" H 4050 2450 50  0001 C CNN
+	1    4050 2450
 	1    0    0    -1
 $EndComp
-Wire Wire Line
-	3700 1800 3600 1800
-Wire Wire Line
-	3600 1800 3600 2100
-Wire Wire Line
-	3600 2100 4350 2100
-Wire Wire Line
-	4350 2100 4350 2000
-Wire Wire Line
-	4350 2000 4300 2000
-Wire Wire Line
-	4300 1800 4400 1800
-Wire Wire Line
-	4400 1800 4400 2150
-Wire Wire Line
-	4400 2150 3700 2150
-Wire Wire Line
-	3700 2150 3700 2000
-Wire Wire Line
-	4600 1800 4550 1800
-Wire Wire Line
-	4550 1800 4550 2100
-Wire Wire Line
-	4550 2100 5250 2100
-Wire Wire Line
-	5250 2100 5250 2000
-Wire Wire Line
-	5250 2000 5200 2000
-Wire Wire Line
-	5200 1800 5300 1800
-Wire Wire Line
-	5300 1800 5300 2150
-Wire Wire Line
-	5300 2150 4500 2150
-Wire Wire Line
-	4500 2150 4500 2000
-Wire Wire Line
-	4500 2000 4600 2000
-Text GLabel 3700 1650 1    50   Input ~ 0
+Text GLabel 3750 1550 0    50   Input ~ 0
 BRRED
-Connection ~ 3700 1800
-Wire Wire Line
-	3700 1650 3700 1800
-Text GLabel 4300 1650 1    50   Input ~ 0
+Text GLabel 4800 1550 2    50   Input ~ 0
 BRGRN
-Wire Wire Line
-	4300 1650 4300 1800
-Connection ~ 4300 1800
-Text GLabel 4600 1650 1    50   Input ~ 0
+Text GLabel 3750 1850 0    50   Input ~ 0
 NRED
-Text GLabel 5200 1650 1    50   Input ~ 0
+Text GLabel 4800 1850 2    50   Input ~ 0
 NGRN
-Wire Wire Line
-	4600 1650 4600 1800
-Connection ~ 4600 1800
-Wire Wire Line
-	5200 1650 5200 1800
-Connection ~ 5200 1800
-Text GLabel 4400 1650 1    50   Input ~ 0
+Text GLabel 4800 1650 2    50   Input ~ 0
 BRGRN2
-Text GLabel 4500 1650 1    50   Input ~ 0
+Text GLabel 3750 1950 0    50   Input ~ 0
 NRED2
-Wire Wire Line
-	4400 1650 4400 1750
-Wire Wire Line
-	4400 1750 4350 1750
-Wire Wire Line
-	4350 1750 4350 1900
-Wire Wire Line
-	4350 1900 4300 1900
-Wire Wire Line
-	4500 1650 4500 1900
-Wire Wire Line
-	4500 1900 4600 1900
-Text GLabel 3700 1900 0    50   Input ~ 0
+Text GLabel 3750 1650 0    50   Input ~ 0
 BRRED2
-Text GLabel 5200 1900 2    50   Input ~ 0
+Text GLabel 4800 1950 2    50   Input ~ 0
 NGRN2
 Text GLabel 4400 950  3    50   Input ~ 0
@@
 Wire Wire Line
 	2850 2200 2850 2300
-Wire Wire Line
-	2850 3100 1950 3100
 Wire Wire Line
 	1950 3100 1950 3700
@@
 	6250 3700 5850 3700
 Wire Wire Line
-	5850 3700 5850 2900
-Wire Wire Line
 	5850 2900 6950 2900
 Wire Wire Line
@@
 Text GLabel 4550 4300 1    50   Input ~ 0
 GND
-$Comp
-L 6PDT:6PDTswitch U?
-U 1 1 5B8F1839
-P 4550 6250
-F 0 "U?" H 4928 7171 50  0000 L CNN
-F 1 "6PDTswitch" H 4928 7080 50  0000 L CNN
-F 2 "" V 4900 6800 50  0001 C CNN
-F 3 "" V 4900 6800 50  0001 C CNN
-	1    4550 6250
-	1    0    0    -1
-$EndComp
 Wire Wire Line
 	2850 1450 2850 1950
@@
 Text GLabel 1850 2200 1    50   Input ~ 0
 BVOUTTRAD
-Text GLabel 4150 5100 1    50   Input ~ 0
+Text GLabel 4150 5150 2    50   Input ~ 0
 BVIN
-Text GLabel 4150 5650 3    50   Input ~ 0
+Text GLabel 3550 5150 0    50   Input ~ 0
 BVOUT
-Text GLabel 4050 5100 1    50   Input ~ 0
+Text GLabel 4150 5050 2    50   Input ~ 0
 BVINTRAD
-Text GLabel 4050 5650 3    50   Input ~ 0
+Text GLabel 3550 5050 0    50   Input ~ 0
 BVOUTTRAD
 Wire Wire Line
-	4250 5100 4250 5000
-Wire Wire Line
-	4250 5000 3900 5000
-Wire Wire Line
-	3900 5000 3900 5700
-Wire Wire Line
-	3900 5700 4250 5700
-Wire Wire Line
-	4250 5700 4250 5650
+	4150 5250 4250 5250
+Wire Wire Line
+	4250 5250 4250 4900
+Wire Wire Line
+	3500 4900 3500 5250
+Wire Wire Line
+	3500 5250 3550 5250
 $Comp
 L 6mmKEMET:KEMET470p5mm U?
@@
 Text GLabel 5900 2050 1    50   Input ~ 0
 NVOUT
-Text GLabel 4450 5100 1    50   Input ~ 0
+Text GLabel 4150 5450 2    50   Input ~ 0
 NVIN
-Text GLabel 4350 5100 1    50   Input ~ 0
+Text GLabel 4150 5350 2    50   Input ~ 0
 NVINTRAD
-Text GLabel 4450 5650 3    50   Input ~ 0
+Text GLabel 3550 5450 0    50   Input ~ 0
 NVOUT
-Text GLabel 4350 5650 3    50   Input ~ 0
+Text GLabel 3550 5350 0    50   Input ~ 0
 NVOUTTRAD
 Wire Wire Line
-	4550 5100 4550 4900
-Wire Wire Line
-	4550 4900 3800 4900
-Wire Wire Line
-	3800 4900 3800 5800
-Wire Wire Line
-	3800 5800 4550 5800
-Wire Wire Line
-	4550 5800 4550 5650
+	4150 5550 4350 5550
+Wire Wire Line
+	4350 5550 4350 4800
+Wire Wire Line
+	3400 4800 3400 5550
+Wire Wire Line
+	3400 5550 3550 5550
+Wire Wire Line
+	3950 1750 3850 1750
+Wire Wire Line
+	3850 1750 3850 1450
+Wire Wire Line
+	3850 1450 4600 1450
+Wire Wire Line
+	4600 1450 4600 1550
+Wire Wire Line
+	4600 1550 4550 1550
+Wire Wire Line
+	4550 1750 4650 1750
+Wire Wire Line
+	4650 1750 4650 1400
+Wire Wire Line
+	4650 1400 3900 1400
+Wire Wire Line
+	3900 1400 3900 1550
+Wire Wire Line
+	3900 1550 3950 1550
+Wire Wire Line
+	3900 1550 3750 1550
+Connection ~ 3900 1550
+Wire Wire Line
+	4800 1550 4600 1550
+Connection ~ 4600 1550
+Wire Wire Line
+	3950 1650 3750 1650
+Wire Wire Line
+	4800 1650 4550 1650
+Wire Wire Line
+	3950 1850 3900 1850
+Wire Wire Line
+	3900 1850 3900 2250
+Wire Wire Line
+	3900 2250 4650 2250
+Wire Wire Line
+	4650 2250 4650 1850
+Wire Wire Line
+	4650 1850 4550 1850
+Wire Wire Line
+	4550 2050 4600 2050
+Wire Wire Line
+	4600 2300 3950 2300
+Wire Wire Line
+	3950 2300 3950 2050
+Wire Wire Line
+	4600 2050 4600 2300
+Wire Wire Line
+	4650 1850 4800 1850
+Connection ~ 4650 1850
+Wire Wire Line
+	3750 1850 3900 1850
+Connection ~ 3900 1850
+Wire Wire Line
+	3750 1950 3950 1950
+Wire Wire Line
+	4800 1950 4550 1950
+$Comp
+L 4pdt:4pdtswitch U?
+U 1 1 5B8E51F2
+P 3650 5950
+F 0 "U?" V 3896 6272 50  0000 R CNN
+F 1 "4pdtswitch" V 3805 6272 50  0000 R CNN
+F 2 "" H 3650 5950 50  0001 C CNN
+F 3 "" H 3650 5950 50  0001 C CNN
+	1    3650 5950
+	1    0    0    -1
+$EndComp
+Wire Wire Line
+	4350 4800 3400 4800
+Wire Wire Line
+	4250 4900 3500 4900
+Text Notes 1600 5350 0    50   ~ 0
+These 2 switches control traditional\nvs 3 band EQ selection
+$Comp
+L 4pdt:4pdtswitch U?
+U 1 1 5B924358
+P 5350 5950
+F 0 "U?" H 5550 6250 50  0000 C CNN
+F 1 "4pdtswitch" H 5550 6150 50  0000 C CNN
+F 2 "" H 5350 5950 50  0001 C CNN
+F 3 "" H 5350 5950 50  0001 C CNN
+	1    5350 5950
+	1    0    0    -1
+$EndComp
+Text GLabel 2850 3100 0    50   Input ~ 0
+BTONE
+Text GLabel 1950 3100 0    50   Input ~ 0
+BTONEIN
+Text GLabel 5850 3700 0    50   Input ~ 0
+NTONEIN
+Text GLabel 5850 2900 0    50   Input ~ 0
+NTONE
+Text GLabel 5250 5150 0    50   Input ~ 0
+BTONE
+Text GLabel 5250 5050 0    50   Input ~ 0
+BTONEIN
+Text GLabel 5850 5050 2    50   Input ~ 0
+NTONEIN
+Text GLabel 5850 5150 2    50   Input ~ 0
+NTONE
 $EndSCHEMATC

Commit message: started updating eeschema
Connections:
- net labels added: OUT
- net labels removed: TOJACK
- wire segments 157 -> 162
Changed lines of the file:
@@
 EELAYER 26 0
 EELAYER END
-$Descr A4 11693 8268
+$Descr B 17000 11000
 encoding utf-8
 Sheet 1 1
@@
 Text GLabel 4450 4300 1    50   Input ~ 0
 NOUT
-Text GLabel 4350 4300 1    50   Input ~ 0
-TOJACK
 Connection ~ 6850 2200
 Wire Wire Line
@@
 Wire Wire Line
 	4800 1950 4550 1950
-$Comp
-L 4pdt:4pdtswitch U?
-U 1 1 5B8E51F2
-P 3650 5950
-F 0 "U?" V 3896 6272 50  0000 R CNN
-F 1 "4pdtswitch" V 3805 6272 50  0000 R CNN
-F 2 "" H 3650 5950 50  0001 C CNN
-F 3 "" H 3650 5950 50  0001 C CNN
-	1    3650 5950
-	1    0    0    -1
-$EndComp
 Wire Wire Line
 	4350 4800 3400 4800
@@
 Text Notes 1600 5350 0    50   ~ 0
 These 2 switches control traditional\nvs 3 band EQ selection
-$Comp
-L 4pdt:4pdtswitch U?
-U 1 1 5B924358
-P 5350 5950
-F 0 "U?" H 5550 6250 50  0000 C CNN
-F 1 "4pdtswitch" H 5550 6150 50  0000 C CNN
-F 2 "" H 5350 5950 50  0001 C CNN
-F 3 "" H 5350 5950 50  0001 C CNN
-	1    5350 5950
-	1    0    0    -1
-$EndComp
 Text GLabel 2850 3100 0    50   Input ~ 0
 BTONE
@@
 Text GLabel 5850 5150 2    50   Input ~ 0
 NTONE
+$Comp
+L 4pdt:4pdtswitch U?
+U 1 1 5B924358
+P 5350 5950
+F 0 "U?" H 5550 6250 50  0000 C CNN
+F 1 "4pdtswitch" H 5550 6150 50  0000 C CNN
+F 2 "" H 5350 5950 50  0001 C CNN
+F 3 "" H 5350 5950 50  0001 C CNN
+	1    5350 5950
+	1    0    0    -1
+$EndComp
+$Comp
+L 4pdt:4pdtswitch U?
+U 1 1 5B8E51F2
+P 3650 5950
+F 0 "U?" H 3900 6250 50  0000 R CNN
+F 1 "4pdtswitch" H 4000 6150 50  0000 R CNN
+F 2 "" H 3650 5950 50  0001 C CNN
+F 3 "" H 3650 5950 50  0001 C CNN
+	1    3650 5950
+	1    0    0    -1
+$EndComp
+Wire Wire Line
+	5250 5350 5200 5350
+Wire Wire Line
+	5200 5350 5200 5800
+Wire Wire Line
+	5200 5800 5900 5800
+Wire Wire Line
+	5900 5800 5900 5350
+Wire Wire Line
+	5900 5350 5850 5350
+Text GLabel 4350 4300 1    50   Input ~ 0
+OUT
 $EndSCHEMATC

Commit message: Finished OD circuit
Parts:
- removed U? (x2): 4pdtswitch, symbol 4pdt:4pdtswitch
- added BT?: Battery, symbol Device:Battery
- added C? (x2): 22n, symbol Device:C
- added C? (x2): 47p, symbol Device:C
- added C? (x3): 10n, symbol Device:C
- added C?: 1n, symbol Device:C
- added C? (x4): 100n, symbol Device:C
- added C?: 47n, symbol Device:C
- added C?: 120p, symbol Device:C
- added C?: 100p, symbol Device:C
- added C?: 4.7n, symbol Device:C
- added C? (x2): 220n, symbol Device:C
- added C?: 2.2n, symbol Device:C
- added C?: 47u, symbol Device:CP1
- added C? (x3): 22u, symbol Device:CP1
- added D? (x4): LED, symbol Device:LED
- added D?: D, symbol Device:D
- added GROUNDBRIDGE: Conn_01x01, symbol Connector_Generic:Conn_01x01
- added Q? (x2): Q_PNP_BCE, symbol Device:Q_PNP_BCE
- added R? (x2): 330k, symbol Device:R
- added R?: 1MEG, symbol Device:R
- added R? (x4): 10k, symbol Device:R
- added R? (x2): 470k, symbol Device:R
- added R?: 39k, symbol Device:R
- added R? (x8): 22k, symbol Device:R
- added R?: 4.7k, symbol Device:R
- added R?: 220k, symbol Device:R
- added R? (x6): 2.2k, symbol Device:R
- added R? (x2): 33k, symbol Device:R
- added R?: 100k, symbol Device:R
- added R?: 3.3K, symbol Device:R
- added R?: 10, symbol Device:R
- added R? (x2): 20k, symbol Device:R
- added R?: 56k, symbol Device:R
- added RV?: 100kREV, symbol Device:R_POT
- added RV?: 100k, symbol Device:R_POT_TRIM
- added RV? (x3): 100k, symbol Device:R_POT
- added U1, U2, U3, U4: TL072, symbol Amplifier_Operational:TL072
- added U? (x2): 6PDTswitch, symbol 6PDT:6PDTswitch
Connections:
- net labels added: 9Vin, 9Vout, BRTONECAPIN, BRTONEGANG1IN, BRTONEGANG1OUT, BRTONEGANG2IN, BTONEGANG1OUT, FinalOut, GAINPOTOUT, GAINSTAGEPOTIN, MASTEROUT, ODVOLIN, ODVOLOUT, ODin, ODout, PRESIN, PRESOUT, SUPPLYIN, Vref, Vref2
- wire segments 162 -> 397

Commit message: started adding footprints
Parts:
- removed RV?: 100k, symbol Device:R_POT
- removed U?: 4pdtswitch, symbol 4pdt:4pdtswitch
- removed U? (x4): KEMET470p5mm, symbol 6mmKEMET:KEMET470p5mm
- removed U?: 3WAYswitch, symbol 3WAY:3WAYswitch
- removed U? (x2): 6PDTswitch, symbol 6PDT:6PDTswitch
- added 3WaySwitch1: Conn_01x04, Pin_Headers:Pin_Header_Straight_1x04_Pitch2.54mm, symbol Connector_Generic:Conn_01x04
- added 4pdt1: Conn_02x06_Counter_Clockwise, symbol Connector_Generic:Conn_02x06_Counter_Clockwise
- added 6pdt1, 6pdt2: Conn_02x09_Odd_Even, symbol Connector_Generic:Conn_02x09_Odd_Even
- added C24, C27: .022u, symbol Device:C
- added C25, C26: 470p, symbol Device:C
- added Jack1: Conn_01x03, Pin_Headers:Pin_Header_Straight_1x03_Pitch2.54mm, symbol Connector_Generic:Conn_01x03
- added R35: 10k, symbol Device:R
- added R?: 250k, symbol Device:R
- added RV?: 50k, symbol Device:R_POT
- BridgeTonePot1: renamed from BridgeTonePot; footprint (none) -> Pin_Headers:Pin_Header_Straight_2x07_Pitch2.54mm
- BridgeVolPot1: renamed from BridgeVolPot; footprint (none) -> Pin_Headers:Pin_Header_Straight_2x07_Pitch2.54mm
- C12: renamed from C?; value 100p -> 220p
- C8: renamed from C?; value 120p -> 220p
- GROUNDBRIDGE1: renamed from GROUNDBRIDGE; footprint (none) -> Pin_Headers:Pin_Header_Straight_1x01_Pitch2.54mm
- NeckTonePot1: renamed from NeckTonePot; footprint (none) -> Pin_Headers:Pin_Header_Straight_2x07_Pitch2.54mm
- NeckVolumePot1: renamed from NeckVolumePot; footprint (none) -> Pin_Headers:Pin_Header_Straight_2x07_Pitch2.54mm
- PickupInputs1: renamed from PickupInputs; footprint (none) -> Pin_Headers:Pin_Header_Straight_1x10_Pitch2.54mm
- R11: renamed from R?; value 56k -> 250k
- R12, R4: renamed from R?; footprint (none) -> Resistors_SMD:R_0603_HandSoldering
- U1, U2, U3, U4: footprint (none) -> Housings_SOIC:SOIC-8_3.9x4.9mm_Pitch1.27mm
- gave numbers to parts that had none: 64
Connections:
- net labels added: ODMIDGND, ODMIDIN, ODMIDOUT, PWRGND
- net labels removed: 9Vin, 9Vout, BTONEGANG1OUT, NWHITE, ODVOLIN, ODVOLOUT, SUPPLYIN
- wire segments 397 -> 419
Other:
- note added: "Ring"
- note added: "Sleeve\n"
- note added: "Tip"

Commit message: Started laying out board
Parts:
- removed BT1: Battery, symbol Device:Battery
- removed C9: 47u, symbol Device:CP1
- removed R6: 39k, symbol Device:R
- added 9V1: Battery, 9vHolder:9vholder, symbol Device:Battery
- added TRANGAIN1: 250k, Potentiometer_THT:Potentiometer_Bourns_3386P_Vertical, symbol Device:R_POT
- added TRBLD1: Conn_02x02_Top_Bottom, TrebBldDIP:TrebBldDIP, symbol Connector_Generic:Conn_02x02_Top_Bottom
- 4pdt1: footprint (none) -> 4pdtFP:4pdtFP
- 6pdt1, 6pdt2: footprint (none) -> 6pdtFP:6pdtFP
- BASS1: renamed from RV4; footprint (none) -> Potentiometer_THT:Potentiometer_Bourns_PTV09A-1_Single_Vertical
- C1, C11, C15, C16, C17, C20, C24, C27, C3, C7: footprint (none) -> Capacitor_SMD:C_1206_3216Metric_Pad1.42x1.75mm_HandSolder
- C10: value 22u -> 100u; footprint (none) -> Capacitor_THT:CP_Radial_D8.0mm_P5.00mm
- C12, C13, C21, C22, C25, C26, C4: footprint (none) -> Capacitor_SMD:C_0805_2012Metric_Pad1.15x1.40mm_HandSolder
- C14, C19: footprint (none) -> Capacitor_THT:CP_Radial_D5.0mm_P2.00mm
- C18, C23: footprint (none) -> Capacitor_SMD:C_2816_7142Metric_Pad3.20x4.45mm_HandSolder
- C2, C6: footprint (none) -> Capacitor_THT:C_Rect_L7.2mm_W4.5mm_P5.00mm_FKS2_FKP2_MKS2_MKP2
- C5: footprint (none) -> Capacitor_SMD:C_1210_3225Metric_Pad1.42x2.65mm_HandSolder
- C8: value 220p -> 470p; footprint (none) -> Capacitor_SMD:C_0805_2012Metric_Pad1.15x1.40mm_HandSolder
- D1, D2, D3, D4, D5: footprint (none) -> LED_THT:LED_D3.0mm
- Q1, Q2: value Q_PNP_BCE -> ZTX951; footprint (none) -> TO_SOT_Packages_THT:TO-92_Inline_Narrow_Oval
- R1, R10, R11, R13, R14, R16, R17, R18, R19, R2, R20, R21, R22, R23, R24, R25, R26, R27, R28, R29, R3, R30, R31, R32, R33, R34, R35, R5, R7, R8, R9: footprint (none) -> Resistor_SMD:R_0805_2012Metric_Pad1.15x1.40mm_HandSolder
- R12, R4: footprint Resistors_SMD:R_0603_HandSoldering -> Resistor_SMD:R_0805_2012Metric_Pad1.15x1.40mm_HandSolder
- R15: value 220k -> 39k; footprint (none) -> Resistor_SMD:R_0805_2012Metric_Pad1.15x1.40mm_HandSolder
- R6: renamed from R?; footprint (none) -> Resistor_SMD:R_0805_2012Metric_Pad1.15x1.40mm_HandSolder
- RANGE1: renamed from RV2; footprint (none) -> Potentiometer_THT:Potentiometer_Bourns_3386P_Vertical
- TIGHT1: renamed from RV1; footprint (none) -> Potentiometer_THT:Potentiometer_Bourns_PTV09A-1_Single_Vertical
- TREBLE1: renamed from RV3; footprint (none) -> Potentiometer_THT:Potentiometer_Bourns_PTV09A-1_Single_Vertical
- VOL1: renamed from RV?; footprint (none) -> Potentiometer_THT:Potentiometer_Bourns_PTV09A-1_Single_Vertical
Connections:
- wire segments 419 -> 437
