File: VolToneEQ/VolToneEQ/VolToneEQ.sch (KiCad schematic (older format))
At the start: 91 parts, among them Q1 ZTX951, Q2 ZTX951, U1 TL072, U2 TL072, U3 TL072, U4 TL072

Commit message: added 100k parallel to volume
Parts:
- added R36: 100k, Resistor_SMD:R_0805_2012Metric_Pad1.15x1.40mm_HandSolder, symbol Device:R
- VOL1: value 50k -> 100k
Connections:
- wire segments 439 -> 444
Changed lines of the file:
@@
 	6250 2100 6200 2100
-Wire Wire Line
-	6200 2100 6200 2000
 Wire Wire Line
 	6200 1650 6350 1650
@@
 Text GLabel 7350 7000 1    50   Input ~ 0
 Vref2
-Text GLabel 6200 2000 0    50   Input ~ 0
+Text GLabel 5600 2000 0    50   Input ~ 0
 ODMIDGND
 Text GLabel 13750 8500 3    50   Input ~ 0
@@
 P 13750 7600
 F 0 "VOL1" H 13680 7554 50  0000 R CNN
-F 1 "50k" H 13680 7645 50  0000 R CNN
+F 1 "100k" H 13680 7645 50  0000 R CNN
 F 2 "Potentiometer_THT:Potentiometer_Bourns_PTV09A-1_Single_Vertical" H 13750 7600 50  0001 C CNN
 F 3 "~" H 13750 7600 50  0001 C CNN
@@
 $EndComp
 Wire Wire Line
-	13750 7750 13750 8400
+	13750 7750 13750 7800
 Connection ~ 13750 8400
 Wire Wire Line
-	13750 7200 13750 7450
+	13750 7200 13750 7400
 Wire Wire Line
 	13900 7600 14100 7600
@@
 PWRGND
 Wire Wire Line
-	6250 2000 6200 2000
+	6200 1650 6200 2100
+Wire Wire Line
+	6250 2000 5600 2000
 Connection ~ 6250 2000
-Connection ~ 6200 2000
-Wire Wire Line
-	6200 2000 6200 1650
+$Comp
+L Device:R R36
+U 1 1 5BB9BC05
+P 13300 7600
+F 0 "R36" H 13370 7646 50  0000 L CNN
+F 1 "100k" H 13300 7450 50  0000 L CNN
+F 2 "Resistor_SMD:R_0805_2012Metric_Pad1.15x1.40mm_HandSolder" V 13230 7600 50  0001 C CNN
+F 3 "~" H 13300 7600 50  0001 C CNN
+	1    13300 7600
+	1    0    0    -1
+$EndComp
+Wire Wire Line
+	13300 7450 13300 7400
+Wire Wire Line
+	13300 7400 13750 7400
+Connection ~ 13750 7400
+Wire Wire Line
+	13750 7400 13750 7450
+Wire Wire Line
+	13300 7750 13300 7800
+Wire Wire Line
+	13300 7800 13750 7800
+Connection ~ 13750 7800
+Wire Wire Line
+	13750 7800 13750 8400
 $EndSCHEMATC
