File: VolToneEQ/VolToneEQ/VolToneEQ.kicad_pcb (KiCad board)
At the start: 2 copper layers, 91 parts, among them Q1 ZTX951, Q2 ZTX951, U1 TL072, U2 TL072, U3 TL072, U4 TL072

Commit message: Organized Layout
Parts:
- C1, C11, C12, C13, C15, C16, C17, C18, C20, C21, C22, C24, C25, C26, C27, C3, C4, C5, C7, C8, R1, R10, R11, R12, R13, R14, R15, R16, R17, R18, R19, R2, R20, R21, R22, R23, R24, R25, R26, R27, R28, R29, R3, R30, R31, R32, R33, R34, R35, R4, R5, R6, R7, R8, R9, U1: moved to B.Cu
- moved GROUNDBRIDGE1 114.6 mm to (86.4, 34.0)
- moved R32 93.1 mm to (87.9, 68.6)
- moved R11 92.4 mm to (79.8, 70.1)
- moved C22 81.0 mm to (74.7, 72.1), turned to 90 degrees
- moved R6 79.5 mm to (95.0, 70.1)
- moved R7 78.6 mm to (127.5, 41.1)
- moved NeckTonePot1 77.4 mm to (146.3, 76.2), turned to 90 degrees
- moved R4 73.6 mm to (129.5, 47.2)
- moved R26 71.0 mm to (124.0, 69.6), turned to 180 degrees
- moved R31 69.0 mm to (104.7, 74.7)
- moved C13 66.4 mm to (153.4, 46.7)
- moved R29 66.0 mm to (141.7, 40.6)
- moved R30 64.7 mm to (147.3, 46.7)
- moved R18 64.0 mm to (138.7, 44.7)
- moved NeckVolumePot1 63.9 mm to (119.9, 78.7)
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Other:
- board outline added: 136.1 x 75.2 mm
