File: VolToneEQ/VolToneEQ/_saved_VolToneEQ.sch (KiCad schematic (older format))
At the start: 91 parts, among them Q1 ZTX951, Q2 ZTX951, U1 TL072, U2 TL072, U3 TL072, U4 TL072

Commit message: routed board
Connections:
- wire segments 439 -> 438
Changed lines of the file:
@@
 	6250 2100 6200 2100
 Wire Wire Line
-	6200 2100 6200 2000
+	6200 2100 6200 1650
 Wire Wire Line
 	6200 1650 6350 1650
@@
 Text GLabel 7350 7000 1    50   Input ~ 0
 Vref2
-Text GLabel 6200 2000 0    50   Input ~ 0
+Text GLabel 6100 2000 0    50   Input ~ 0
 ODMIDGND
 Text GLabel 13750 8500 3    50   Input ~ 0
@@
 PWRGND
 Wire Wire Line
-	6250 2000 6200 2000
+	6250 2000 6100 2000
 Connection ~ 6250 2000
-Connection ~ 6200 2000
-Wire Wire Line
-	6200 2000 6200 1650
 $EndSCHEMATC
